Commit message: add timestamp adjust and timestamp reverse function in msg_conversion.cc

File: cartographer_ros/urdf/gazebo.urdf (robot description, URDF)
Before this commit: robot movexbot, 4 links, 3 joints
Links:
- removed link footprint
- removed link hokuyo_link
- removed link lidar_link
- added link base_link
- added link laser_link
- added link odom_link
Joints:
- removed joint hokuyo_link
- removed joint lidar_link
- added joint base_link: type fixed, parent odom_link, child base_link, origin xyz=0.075 0 0.0 rpy=0 0 0
- added joint laser_link: type fixed, parent base_link, child laser_link, origin xyz=0.0 0 0.0 rpy=0 0 0
- joint imu_link: parent footprint -> base_link
