Commit message: modified glog settings update movexbot_simulation.launch

File: cartographer_ros/urdf/demo.urdf (robot description, URDF)
Before this commit: robot movexbot, 4 links, 3 joints
Links:
- removed link imu_link
- removed link laser_link
- added link gyro_link
- added link laser_link_horizontal
Joints:
- removed joint base_link
- removed joint imu_link
- removed joint laser_link
- added joint base_link_joint: type fixed, parent odom_link, child base_link, origin xyz=0.0 0 0
- added joint gyro_link_joint: type fixed, parent base_link, child gyro_link, origin xyz=0 0 0
- added joint laser_link_horizontal: type fixed, parent base_link, child laser_link_horizontal, origin xyz=0.3035 0 0.0 rpy=0 0 0
